File: meas-tensio.kicad_pcb (KiCad board)
At the start: 2 copper layers, 100 x 100 mm, 43 parts, among them J1 Tens4, J2 Tens3, J3 Tens2, J4 Tens1, J6 CAN1, J7 CAN2, P1 CONN_PROG+SER_AVR, Q1 BSS83P, U1 ATMEGA168PA-AU, U2 MCP2515-E/SO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

Commit message: Fix edge
Other:
- board size 100 x 100 mm -> 77.5 x 47 mm
Changed lines of the file:
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@@
   )
   (page A4)
+  (title_block
+    (title "Tensiometer measurement board")
+    (company "Klaus Schneider-Zapp")
+  )
   (layers
     (0 F.Cu signal)
@@
     )
   )
+  (gr_line (start 280.67 111.76) (end 203.2 111.76) (angle 90) (layer Edge.Cuts) (width 0.1))
+  (gr_line (start 280.67 158.75) (end 280.67 111.76) (angle 90) (layer Edge.Cuts) (width 0.1))
+  (gr_line (start 203.2 158.75) (end 203.2 111.76) (angle 90) (layer Edge.Cuts) (width 0.1))
+  (gr_line (start 280.67 158.75) (end 203.2 158.75) (angle 90) (layer Edge.Cuts) (width 0.1))
   (gr_text "2018 KSZ" (at 212.725 155.575) (layer B.Cu)
     (effects (font (size 1.5 1.5) (thickness 0.3)) (justify mirror))
@@
     (effects (font (size 1.5 1.5) (thickness 0.3)))
   )
-  (gr_line (start 180 60) (end 180 160) (angle 90) (layer Edge.Cuts) (width 0.1))
-  (gr_line (start 280 60) (end 180 60) (angle 90) (layer Edge.Cuts) (width 0.1))
-  (gr_line (start 280 160) (end 280 60) (angle 90) (layer Edge.Cuts) (width 0.1))
-  (gr_line (start 180 160) (end 280 160) (angle 90) (layer Edge.Cuts) (width 0.1))
   (segment (start 232.80116 134.38378) (end 230.512572 134.38378) (width 0.508) (layer B.Cu) (net 1) (status 400000))
   (segment (start 227.965 131.836208) (end 227.965 131.826) (width 0.508) (layer B.Cu) (net 1))

Commit message: Improve analogue part
Parts:
- added C13: 10n, Capacitor_SMD:C_0805_2012Metric, B.Cu at (271.8, 130.6)
- moved JP2 40.1 mm to (275.6, 124.2), turned to 90 degrees
- moved JP1 3.60 mm to (239.3, 146.6)
- moved U7 1.91 mm to (266.7, 125.7)
- moved Q1 1.78 mm to (271.3, 123.3)
- moved R5 1.78 mm to (275.2, 123.3)
- moved C3 1.78 mm to (270.6, 119.5)
- moved R8 1.78 mm to (273.7, 119.5)
Connections:
- JP2 pad 1: Net-(C3-Pad1) -> Net-(J1-Pad3)
- JP2 pad 2: Net-(J1-Pad3) -> Net-(C3-Pad1)
- U6 pad 8: Net-(C3-Pad1) -> /12V
- U8 pad 14: Net-(C3-Pad1) -> /12V
Routing:
- net /12V: track 61.8 -> 122.8 mm, vias 0 -> 3
- net Net-(C3-Pad1): track 64.0 -> 16.0 mm, vias 2 -> 0
- net Net-(J1-Pad3): track 73.9 -> 96.3 mm
- net GNDA: track 315.7 -> 324.9 mm
- net Net-(JP1-Pad2): track 15.5 -> 19.5 mm
- net Net-(U1-Pad24): track 59.9 -> 63.4 mm
- net Net-(U1-Pad26): track 73.1 -> 76.4 mm
- net Net-(U1-Pad25): track 51.9 -> 54.4 mm
- net Net-(R6-Pad1): track 16.2 -> 18.1 mm
- net Net-(JP4-Pad2): track 32.0 -> 30.3 mm
- net Net-(R8-Pad1): track 120.7 -> 119.7 mm
